File: trimux/trimuxIO/trimuxIO.sch (KiCad schematic (older format))
At the start: 12 parts, among them J1 SP3T, J2 SP3T, P1 IO, P2 I, Q1 2n3906, Q2 2n3904

Commit message: IO
Parts:
- added D1(2)2, D1(2)3, D1(2)4, D1(2)5, D1(2)6, D1(2)7, D1(2)8, D1(2)9: LED_Dual_2pin, LEDs:LED_D5.0mm, symbol LED_Dual_2pin
- added J10, J3, J4, J5, J6, J7, J8, J9: SP3T, trimuxIO:Pin_Header_Straight_1x04_Pitch3.10mm, symbol SP3T
- added P10, P11, P4, P5, P6, P7, P8, P9: IO, Pin_Headers:Pin_Header_Straight_1x01_Pitch2.54mm, symbol CONN_01X01
- added P3: CONN_01X03, Pin_Headers:Pin_Header_Straight_1x03_Pitch2.54mm, symbol CONN_01X03
- added Q10, Q12, Q14, Q16, Q18, Q4, Q6, Q8: 2n3906, TO_SOT_Packages_THT:TO-92_Inline_Wide, symbol Q_PNP_EBC
- added Q11, Q13, Q15, Q17, Q3, Q5, Q7, Q9: 2n3904, TO_SOT_Packages_THT:TO-92_Inline_Wide, symbol Q_NPN_EBC
- added R10, R11, R18, R19, R20, R27, R28, R29: 1k, Resistors_THT:R_Axial_DIN0411_L9.9mm_D3.6mm_P15.24mm_Horizontal, symbol R
- added R12, R13, R14, R21, R22, R23, R6, R7: 150, Resistors_THT:R_Axial_DIN0411_L9.9mm_D3.6mm_P15.24mm_Horizontal, symbol R
- added R15, R16, R17, R24, R25, R26, R8, R9: 15k, Resistors_THT:R_Axial_DIN0411_L9.9mm_D3.6mm_P15.24mm_Horizontal, symbol R
- J1, J2: footprint trimuxIO:Pin_Header_Straight_1x04_Pitch3.00mm -> trimuxIO:Pin_Header_Straight_1x04_Pitch3.10mm
- Q1, Q2: footprint TO_SOT_Packages_THT:TO-92_Molded_Narrow -> TO_SOT_Packages_THT:TO-92_Inline_Wide
Connections:
- net labels added: GNDREF
- net labels removed: Earth
- wire segments 27 -> 228
Other:
- moved on the sheet: D1(2)1, J1, J2, P1, P2, Q1, Q2, R1, R2, R3, R4, R5
