File: trimux/trimuxIO/trimuxIO.kicad_pcb (KiCad board)
At the start: 2 copper layers, 12 parts, among them J1 SP3T, J2 SP3T, P1 IO, P2 I, Q1 2n3906, Q2 2n3904

Commit message: IO
Parts:
- removed J2: SP3T, trimuxIO:Pin_Header_Straight_1x04_Pitch3.00mm
- removed P2: I, Pin_Headers:Pin_Header_Straight_1x01_Pitch2.54mm
- removed R1: 15k, Resistors_THT:R_Axial_DIN0411_L9.9mm_D3.6mm_P15.24mm_Horizontal
- removed R5: 150, Resistors_THT:R_Axial_DIN0411_L9.9mm_D3.6mm_P15.24mm_Horizontal
- added D1(2)2: LED_Dual_2pin, LEDs:LED_D5.0mm, F.Cu at (131.4, 140.3)
- added D1(2)3: LED_Dual_2pin, LEDs:LED_D5.0mm, F.Cu at (85.7, 140.3)
- added D1(2)4: LED_Dual_2pin, LEDs:LED_D5.0mm, F.Cu at (146.7, 140.3)
- added D1(2)5: LED_Dual_2pin, LEDs:LED_D5.0mm, F.Cu at (55.9, 140.3)
- added D1(2)6: LED_Dual_2pin, LEDs:LED_D5.0mm, F.Cu at (101.0, 140.3)
- added D1(2)7: LED_Dual_2pin, LEDs:LED_D5.0mm, F.Cu at (161.9, 140.3)
- added D1(2)8: LED_Dual_2pin, LEDs:LED_D5.0mm, F.Cu at (70.5, 140.3)
- added D1(2)9: LED_Dual_2pin, LEDs:LED_D5.0mm, F.Cu at (116.2, 140.3)
- added J10: SP3T, trimuxIO:Pin_Header_Straight_1x04_Pitch3.10mm, F.Cu at (113.0, 106.7)
- added J3: SP3T, trimuxIO:Pin_Header_Straight_1x04_Pitch3.10mm, F.Cu at (128.3, 106.7)
- added J4: SP3T, trimuxIO:Pin_Header_Straight_1x04_Pitch3.10mm, F.Cu at (82.5, 106.7)
- added J5: SP3T, trimuxIO:Pin_Header_Straight_1x04_Pitch3.10mm, F.Cu at (143.5, 106.7)
- added J6: SP3T, trimuxIO:Pin_Header_Straight_1x04_Pitch3.10mm, F.Cu at (52.1, 106.7)
- added J7: SP3T, trimuxIO:Pin_Header_Straight_1x04_Pitch3.10mm, F.Cu at (97.8, 106.7)
- added J8: SP3T, trimuxIO:Pin_Header_Straight_1x04_Pitch3.10mm, F.Cu at (158.8, 106.7)
- added J9: SP3T, trimuxIO:Pin_Header_Straight_1x04_Pitch3.10mm, F.Cu at (67.3, 106.7)
- added P10: IO, Pin_Headers:Pin_Header_Straight_1x01_Pitch2.54mm, F.Cu at (94.0, 68.6)
- added P11: IO, Pin_Headers:Pin_Header_Straight_1x01_Pitch2.54mm, F.Cu at (101.6, 68.6)
- added P3: CONN_01X03, Pin_Headers:Pin_Header_Straight_1x03_Pitch2.54mm, F.Cu at (36.8, 76.2)
- added P4: IO, Pin_Headers:Pin_Header_Straight_1x01_Pitch2.54mm, F.Cu at (104.1, 68.6)
- added P5: IO, Pin_Headers:Pin_Header_Straight_1x01_Pitch2.54mm, F.Cu at (96.5, 68.6)
- added P6: IO, Pin_Headers:Pin_Header_Straight_1x01_Pitch2.54mm, F.Cu at (106.7, 68.6)
- added P7: IO, Pin_Headers:Pin_Header_Straight_1x01_Pitch2.54mm, F.Cu at (91.4, 68.6)
- added P8: IO, Pin_Headers:Pin_Header_Straight_1x01_Pitch2.54mm, F.Cu at (99.1, 68.6)
- added P9: IO, Pin_Headers:Pin_Header_Straight_1x01_Pitch2.54mm, F.Cu at (109.2, 68.6)
- added Q10: 2n3906, TO_SOT_Packages_THT:TO-92_Inline_Wide, F.Cu at (54.6, 101.6)
- added Q11: 2n3904, TO_SOT_Packages_THT:TO-92_Inline_Wide, F.Cu at (100.3, 95.2)
- added Q12: 2n3906, TO_SOT_Packages_THT:TO-92_Inline_Wide, F.Cu at (100.3, 101.6)
- added Q13: 2n3904, TO_SOT_Packages_THT:TO-92_Inline_Wide, F.Cu at (161.3, 95.2)
- added Q14: 2n3906, TO_SOT_Packages_THT:TO-92_Inline_Wide, F.Cu at (161.3, 101.6)
- added Q15: 2n3904, TO_SOT_Packages_THT:TO-92_Inline_Wide, F.Cu at (69.8, 95.2)
- added Q16: 2n3906, TO_SOT_Packages_THT:TO-92_Inline_Wide, F.Cu at (69.8, 101.6)
- added Q17: 2n3904, TO_SOT_Packages_THT:TO-92_Inline_Wide, F.Cu at (115.6, 95.2)
- added Q18: 2n3906, TO_SOT_Packages_THT:TO-92_Inline_Wide, F.Cu at (115.6, 101.6)
- added Q3: 2n3904, TO_SOT_Packages_THT:TO-92_Inline_Wide, F.Cu at (130.8, 95.2)
- added Q4: 2n3906, TO_SOT_Packages_THT:TO-92_Inline_Wide, F.Cu at (130.8, 101.6)
- added Q5: 2n3904, TO_SOT_Packages_THT:TO-92_Inline_Wide, F.Cu at (85.1, 95.2)
- added Q6: 2n3906, TO_SOT_Packages_THT:TO-92_Inline_Wide, F.Cu at (85.1, 101.6)
- added Q7: 2n3904, TO_SOT_Packages_THT:TO-92_Inline_Wide, F.Cu at (146.1, 95.2)
- added Q8: 2n3906, TO_SOT_Packages_THT:TO-92_Inline_Wide, F.Cu at (146.1, 101.6)
- added Q9: 2n3904, TO_SOT_Packages_THT:TO-92_Inline_Wide, F.Cu at (54.6, 95.2)
- added R10: 1k, Resistors_THT:R_Axial_DIN0411_L9.9mm_D3.6mm_P15.24mm_Horizontal, F.Cu at (132.1, 134.6)
- added R11: 1k, Resistors_THT:R_Axial_DIN0411_L9.9mm_D3.6mm_P15.24mm_Horizontal, F.Cu at (86.4, 134.6)
- added R12: 150, Resistors_THT:R_Axial_DIN0411_L9.9mm_D3.6mm_P15.24mm_Horizontal, F.Cu at (142.2, 90.4)
- added R13: 150, Resistors_THT:R_Axial_DIN0411_L9.9mm_D3.6mm_P15.24mm_Horizontal, F.Cu at (50.8, 90.4)
- added R14: 150, Resistors_THT:R_Axial_DIN0411_L9.9mm_D3.6mm_P15.24mm_Horizontal, F.Cu at (96.5, 90.4)
- added R15: 15k, Resistors_THT:R_Axial_DIN0411_L9.9mm_D3.6mm_P15.24mm_Horizontal, F.Cu at (141.6, 127.0)
- added R16: 15k, Resistors_THT:R_Axial_DIN0411_L9.9mm_D3.6mm_P15.24mm_Horizontal, F.Cu at (50.3, 127.0)
- added R17: 15k, Resistors_THT:R_Axial_DIN0411_L9.9mm_D3.6mm_P15.24mm_Horizontal, F.Cu at (95.9, 127.0)
- added R18: 1k, Resistors_THT:R_Axial_DIN0411_L9.9mm_D3.6mm_P15.24mm_Horizontal, F.Cu at (147.3, 134.6)
- added R19: 1k, Resistors_THT:R_Axial_DIN0411_L9.9mm_D3.6mm_P15.24mm_Horizontal, F.Cu at (55.9, 134.6)
- added R20: 1k, Resistors_THT:R_Axial_DIN0411_L9.9mm_D3.6mm_P15.24mm_Horizontal, F.Cu at (101.6, 134.6)
- added R21: 150, Resistors_THT:R_Axial_DIN0411_L9.9mm_D3.6mm_P15.24mm_Horizontal, F.Cu at (157.5, 90.4)
- added R22: 150, Resistors_THT:R_Axial_DIN0411_L9.9mm_D3.6mm_P15.24mm_Horizontal, F.Cu at (66.0, 90.4)
- added R23: 150, Resistors_THT:R_Axial_DIN0411_L9.9mm_D3.6mm_P15.24mm_Horizontal, F.Cu at (111.8, 90.4)
- added R24: 15k, Resistors_THT:R_Axial_DIN0411_L9.9mm_D3.6mm_P15.24mm_Horizontal, F.Cu at (156.8, 127.0)
- added R25: 15k, Resistors_THT:R_Axial_DIN0411_L9.9mm_D3.6mm_P15.24mm_Horizontal, F.Cu at (65.4, 127.0)
- added R26: 15k, Resistors_THT:R_Axial_DIN0411_L9.9mm_D3.6mm_P15.24mm_Horizontal, F.Cu at (111.1, 127.0)
- added R27: 1k, Resistors_THT:R_Axial_DIN0411_L9.9mm_D3.6mm_P15.24mm_Horizontal, F.Cu at (162.6, 134.6)
- added R28: 1k, Resistors_THT:R_Axial_DIN0411_L9.9mm_D3.6mm_P15.24mm_Horizontal, F.Cu at (71.1, 134.6)
- added R29: 1k, Resistors_THT:R_Axial_DIN0411_L9.9mm_D3.6mm_P15.24mm_Horizontal, F.Cu at (116.8, 134.6)
- added R6: 150, Resistors_THT:R_Axial_DIN0411_L9.9mm_D3.6mm_P15.24mm_Horizontal, F.Cu at (127.0, 90.4)
- added R7: 150, Resistors_THT:R_Axial_DIN0411_L9.9mm_D3.6mm_P15.24mm_Horizontal, F.Cu at (81.3, 90.4)
- added R8: 15k, Resistors_THT:R_Axial_DIN0411_L9.9mm_D3.6mm_P15.24mm_Horizontal, F.Cu at (126.4, 127.0)
- added R9: 15k, Resistors_THT:R_Axial_DIN0411_L9.9mm_D3.6mm_P15.24mm_Horizontal, F.Cu at (80.6, 127.0)
- J1: footprint trimuxIO:Pin_Header_Straight_1x04_Pitch3.00mm -> trimuxIO:Pin_Header_Straight_1x04_Pitch3.10mm
- Q1, Q2: footprint TO_SOT_Packages_THT:TO-92_Molded_Narrow -> TO_SOT_Packages_THT:TO-92_Inline_Wide
- moved R2 108.8 mm to (34.9, 127.0), turned to 270 degrees
- moved D1(2)1 108.0 mm to (40.0, 140.3)
- moved R3 105.2 mm to (40.6, 134.6), turned to 90 degrees
- moved Q2 86.4 mm to (39.4, 95.2), turned to 180 degrees
- moved J1 82.6 mm to (36.8, 106.7)
- moved Q1 78.0 mm to (39.4, 101.6), turned to 180 degrees
- moved R4 76.1 mm to (35.6, 90.4), turned to 45 degrees
- moved P1 36.9 mm to (88.9, 68.6)
Connections:
- D1(2)1 pad 1: Net-(D1(2)1-Pad1) -> GNDREF
- J1 pad 3: Net-(J1-Pad3) -> Net-(J1-Pad1)
- R2 pad 2: Earth -> GNDREF
Routing:
- net +5V: track 0.00 -> 722.4 mm
- net -5V: track 0.00 -> 546.5 mm
- net GNDREF: track 0.00 -> 230.1 mm
- net Net-(P9-Pad1): track 0.00 -> 53.4 mm
- net Net-(P1-Pad1): track 0.00 -> 50.3 mm
- net Net-(J7-Pad1): track 0.00 -> 44.1 mm
- net Net-(J8-Pad1): track 0.00 -> 44.1 mm
- net Net-(J3-Pad1): track 0.00 -> 44.1 mm
- net Net-(J9-Pad1): track 0.00 -> 44.1 mm
- net Net-(J6-Pad1): track 0.00 -> 44.1 mm
- net Net-(J10-Pad1): track 0.00 -> 44.1 mm
- net Net-(J4-Pad1): track 0.00 -> 44.1 mm
- net Net-(J1-Pad1): track 0.00 -> 44.1 mm
- net Net-(J5-Pad1): track 0.00 -> 44.1 mm
- net Net-(P6-Pad1): track 0.00 -> 40.3 mm
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Other:
- net class Default: clearance 0.2 -> 0.4; trace_width 0.25 -> 1.27
- rule trace_clearance: 0.2 -> 0.4

Commit message: IO
Parts:
- added D1(2)1: LED_Dual_2pin, LEDs:LED_D5.0mm, F.Cu at (245.1, 160.0)
- added D1(2)2: LED_Dual_2pin, LEDs:LED_D5.0mm, F.Cu at (245.1, 68.6)
- added D1(2)3: LED_Dual_2pin, LEDs:LED_D5.0mm, F.Cu at (245.1, 114.3)
- added D1(2)4: LED_Dual_2pin, LEDs:LED_D5.0mm, F.Cu at (245.1, 53.3)
- added D1(2)5: LED_Dual_2pin, LEDs:LED_D5.0mm, F.Cu at (245.1, 144.1)
- added D1(2)6: LED_Dual_2pin, LEDs:LED_D5.0mm, F.Cu at (245.1, 99.1)
- added D1(2)7: LED_Dual_2pin, LEDs:LED_D5.0mm, F.Cu at (245.1, 38.1)
- added D1(2)8: LED_Dual_2pin, LEDs:LED_D5.0mm, F.Cu at (245.1, 129.5)
- added D1(2)9: LED_Dual_2pin, LEDs:LED_D5.0mm, F.Cu at (245.1, 83.8)
- added J1: SP3T, trimuxIO:Pin_Header_Straight_1x04_Pitch3.10mm, F.Cu at (211.5, 163.2)
- added J10: SP3T, trimuxIO:Pin_Header_Straight_1x04_Pitch3.10mm, F.Cu at (211.5, 87.0)
- added J3: SP3T, trimuxIO:Pin_Header_Straight_1x04_Pitch3.10mm, F.Cu at (211.5, 71.8)
- added J4: SP3T, trimuxIO:Pin_Header_Straight_1x04_Pitch3.10mm, F.Cu at (211.5, 117.5)
- added J5: SP3T, trimuxIO:Pin_Header_Straight_1x04_Pitch3.10mm, F.Cu at (211.5, 56.5)
- added J6: SP3T, trimuxIO:Pin_Header_Straight_1x04_Pitch3.10mm, F.Cu at (211.5, 148.0)
- added J7: SP3T, trimuxIO:Pin_Header_Straight_1x04_Pitch3.10mm, F.Cu at (211.5, 102.2)
- added J8: SP3T, trimuxIO:Pin_Header_Straight_1x04_Pitch3.10mm, F.Cu at (211.5, 41.3)
- added J9: SP3T, trimuxIO:Pin_Header_Straight_1x04_Pitch3.10mm, F.Cu at (211.5, 132.7)
- added P1: IO, Pin_Headers:Pin_Header_Straight_1x01_Pitch2.54mm, F.Cu at (173.4, 111.1)
- added P10: IO, Pin_Headers:Pin_Header_Straight_1x01_Pitch2.54mm, F.Cu at (173.4, 106.0)
- added P11: IO, Pin_Headers:Pin_Header_Straight_1x01_Pitch2.54mm, F.Cu at (173.4, 98.4)
- added P3: CONN_01X03, Pin_Headers:Pin_Header_Straight_1x03_Pitch2.54mm, F.Cu at (181.0, 163.2)
- added P4: IO, Pin_Headers:Pin_Header_Straight_1x01_Pitch2.54mm, F.Cu at (173.4, 95.9)
- added P5: IO, Pin_Headers:Pin_Header_Straight_1x01_Pitch2.54mm, F.Cu at (173.4, 103.5)
- added P6: IO, Pin_Headers:Pin_Header_Straight_1x01_Pitch2.54mm, F.Cu at (173.4, 93.3)
- added P7: IO, Pin_Headers:Pin_Header_Straight_1x01_Pitch2.54mm, F.Cu at (173.4, 108.6)
- added P8: IO, Pin_Headers:Pin_Header_Straight_1x01_Pitch2.54mm, F.Cu at (173.4, 101.0)
- added P9: IO, Pin_Headers:Pin_Header_Straight_1x01_Pitch2.54mm, F.Cu at (173.4, 90.8)
- added Q1: 2n3906, TO_SOT_Packages_THT:TO-92_Inline_Wide, F.Cu at (206.4, 160.7)
- added Q10: 2n3906, TO_SOT_Packages_THT:TO-92_Inline_Wide, F.Cu at (206.4, 145.4)
- added Q11: 2n3904, TO_SOT_Packages_THT:TO-92_Inline_Wide, F.Cu at (200.0, 99.7)
- added Q12: 2n3906, TO_SOT_Packages_THT:TO-92_Inline_Wide, F.Cu at (206.4, 99.7)
- added Q13: 2n3904, TO_SOT_Packages_THT:TO-92_Inline_Wide, F.Cu at (200.0, 38.7)
- added Q14: 2n3906, TO_SOT_Packages_THT:TO-92_Inline_Wide, F.Cu at (206.4, 38.7)
- added Q15: 2n3904, TO_SOT_Packages_THT:TO-92_Inline_Wide, F.Cu at (200.0, 130.2)
- added Q16: 2n3906, TO_SOT_Packages_THT:TO-92_Inline_Wide, F.Cu at (206.4, 130.2)
- added Q17: 2n3904, TO_SOT_Packages_THT:TO-92_Inline_Wide, F.Cu at (200.0, 84.5)
- added Q18: 2n3906, TO_SOT_Packages_THT:TO-92_Inline_Wide, F.Cu at (206.4, 84.5)
- added Q2: 2n3904, TO_SOT_Packages_THT:TO-92_Inline_Wide, F.Cu at (200.0, 160.7)
- added Q3: 2n3904, TO_SOT_Packages_THT:TO-92_Inline_Wide, F.Cu at (200.0, 69.2)
- added Q4: 2n3906, TO_SOT_Packages_THT:TO-92_Inline_Wide, F.Cu at (206.4, 69.2)
- added Q5: 2n3904, TO_SOT_Packages_THT:TO-92_Inline_Wide, F.Cu at (200.0, 114.9)
- added Q6: 2n3906, TO_SOT_Packages_THT:TO-92_Inline_Wide, F.Cu at (206.4, 114.9)
- added Q7: 2n3904, TO_SOT_Packages_THT:TO-92_Inline_Wide, F.Cu at (200.0, 54.0)
- added Q8: 2n3906, TO_SOT_Packages_THT:TO-92_Inline_Wide, F.Cu at (206.4, 54.0)
- added Q9: 2n3904, TO_SOT_Packages_THT:TO-92_Inline_Wide, F.Cu at (200.0, 145.4)
- added R10: 1k, Resistors_THT:R_Axial_DIN0411_L9.9mm_D3.6mm_P15.24mm_Horizontal, F.Cu at (239.4, 67.9)
- added R11: 1k, Resistors_THT:R_Axial_DIN0411_L9.9mm_D3.6mm_P15.24mm_Horizontal, F.Cu at (239.4, 113.7)
- added R12: 150, Resistors_THT:R_Axial_DIN0411_L9.9mm_D3.6mm_P15.24mm_Horizontal, F.Cu at (195.2, 57.8)
- added R13: 150, Resistors_THT:R_Axial_DIN0411_L9.9mm_D3.6mm_P15.24mm_Horizontal, F.Cu at (195.2, 149.2)
- added R14: 150, Resistors_THT:R_Axial_DIN0411_L9.9mm_D3.6mm_P15.24mm_Horizontal, F.Cu at (195.2, 103.5)
- added R15: 15k, Resistors_THT:R_Axial_DIN0411_L9.9mm_D3.6mm_P15.24mm_Horizontal, F.Cu at (231.8, 58.4)
- added R16: 15k, Resistors_THT:R_Axial_DIN0411_L9.9mm_D3.6mm_P15.24mm_Horizontal, F.Cu at (231.8, 149.7)
- added R17: 15k, Resistors_THT:R_Axial_DIN0411_L9.9mm_D3.6mm_P15.24mm_Horizontal, F.Cu at (231.8, 104.1)
- added R18: 1k, Resistors_THT:R_Axial_DIN0411_L9.9mm_D3.6mm_P15.24mm_Horizontal, F.Cu at (239.4, 52.7)
- added R19: 1k, Resistors_THT:R_Axial_DIN0411_L9.9mm_D3.6mm_P15.24mm_Horizontal, F.Cu at (239.4, 144.1)
- added R2: 15k, Resistors_THT:R_Axial_DIN0411_L9.9mm_D3.6mm_P15.24mm_Horizontal, F.Cu at (231.8, 165.1)
- added R20: 1k, Resistors_THT:R_Axial_DIN0411_L9.9mm_D3.6mm_P15.24mm_Horizontal, F.Cu at (239.4, 98.4)
- added R21: 150, Resistors_THT:R_Axial_DIN0411_L9.9mm_D3.6mm_P15.24mm_Horizontal, F.Cu at (195.2, 42.5)
- added R22: 150, Resistors_THT:R_Axial_DIN0411_L9.9mm_D3.6mm_P15.24mm_Horizontal, F.Cu at (195.2, 134.0)
- added R23: 150, Resistors_THT:R_Axial_DIN0411_L9.9mm_D3.6mm_P15.24mm_Horizontal, F.Cu at (195.2, 88.3)
- added R24: 15k, Resistors_THT:R_Axial_DIN0411_L9.9mm_D3.6mm_P15.24mm_Horizontal, F.Cu at (231.8, 43.2)
- added R25: 15k, Resistors_THT:R_Axial_DIN0411_L9.9mm_D3.6mm_P15.24mm_Horizontal, F.Cu at (231.8, 134.6)
- added R26: 15k, Resistors_THT:R_Axial_DIN0411_L9.9mm_D3.6mm_P15.24mm_Horizontal, F.Cu at (231.8, 88.9)
- added R27: 1k, Resistors_THT:R_Axial_DIN0411_L9.9mm_D3.6mm_P15.24mm_Horizontal, F.Cu at (239.4, 37.5)
- added R28: 1k, Resistors_THT:R_Axial_DIN0411_L9.9mm_D3.6mm_P15.24mm_Horizontal, F.Cu at (239.4, 128.9)
- added R29: 1k, Resistors_THT:R_Axial_DIN0411_L9.9mm_D3.6mm_P15.24mm_Horizontal, F.Cu at (239.4, 83.2)
- added R3: 1k, Resistors_THT:R_Axial_DIN0411_L9.9mm_D3.6mm_P15.24mm_Horizontal, F.Cu at (239.4, 159.4)
- added R4: 150, Resistors_THT:R_Axial_DIN0411_L9.9mm_D3.6mm_P15.24mm_Horizontal, F.Cu at (195.2, 164.5)
- added R6: 150, Resistors_THT:R_Axial_DIN0411_L9.9mm_D3.6mm_P15.24mm_Horizontal, F.Cu at (195.2, 73.0)
- added R7: 150, Resistors_THT:R_Axial_DIN0411_L9.9mm_D3.6mm_P15.24mm_Horizontal, F.Cu at (195.2, 118.7)
- added R8: 15k, Resistors_THT:R_Axial_DIN0411_L9.9mm_D3.6mm_P15.24mm_Horizontal, F.Cu at (231.8, 73.7)
- added R9: 15k, Resistors_THT:R_Axial_DIN0411_L9.9mm_D3.6mm_P15.24mm_Horizontal, F.Cu at (231.8, 119.4)
- moved D1(2)7 117.0 mm to (111.1, 34.9), turned to 90 degrees
- moved R27 115.5 mm to (105.4, 34.3), turned to 180 degrees
- moved Q13 112.4 mm to (66.0, 35.6), turned to 270 degrees
- moved Q14 110.7 mm to (72.4, 35.6), turned to 270 degrees
- moved R21 109.0 mm to (61.2, 39.4), turned to 180 degrees
- moved J8 106.3 mm to (77.5, 38.1), turned to 90 degrees
- moved R24 105.1 mm to (97.8, 40.0), turned to 0 degrees
- moved D1(2)4 96.9 mm to (111.1, 50.2), turned to 90 degrees
- moved R18 94.9 mm to (105.4, 49.5), turned to 180 degrees
- moved Q7 91.5 mm to (66.0, 50.8), turned to 270 degrees
- moved Q8 89.5 mm to (72.4, 50.8), turned to 270 degrees
- moved R12 88.6 mm to (61.2, 54.6), turned to 180 degrees
- moved J5 84.9 mm to (77.5, 53.3), turned to 90 degrees
- moved P3 84.4 mm to (47.0, 160.0), turned to 270 degrees
- moved R15 84.1 mm to (97.8, 55.2), turned to 0 degrees
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Routing:
- net +5V: track 722.4 -> 1444.8 mm
- net -5V: track 546.5 -> 1092.9 mm
- net GNDREF: track 230.1 -> 460.3 mm
- net Net-(P9-Pad1): track 53.4 -> 106.8 mm
- net Net-(P1-Pad1): track 50.3 -> 100.5 mm
- net Net-(J5-Pad1): track 44.1 -> 88.3 mm
- net Net-(J4-Pad1): track 44.1 -> 88.3 mm
- net Net-(J10-Pad1): track 44.1 -> 88.3 mm
- net Net-(J3-Pad1): track 44.1 -> 88.3 mm
- net Net-(J1-Pad1): track 44.1 -> 88.3 mm
- net Net-(J9-Pad1): track 44.1 -> 88.3 mm
- net Net-(J8-Pad1): track 44.1 -> 88.3 mm
- net Net-(J6-Pad1): track 44.1 -> 88.3 mm
- net Net-(J7-Pad1): track 44.1 -> 88.3 mm
- net Net-(P6-Pad1): track 40.3 -> 80.6 mm
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
Commit message: half-adder
Parts:
- removed the D1(2)1 at (245.1, 160.0)
- removed the D1(2)2 at (245.1, 68.6)
- removed the D1(2)3 at (245.1, 114.3)
- removed the D1(2)4 at (245.1, 53.3)
- removed the D1(2)5 at (245.1, 144.1)
- removed the D1(2)6 at (245.1, 99.1)
- removed the D1(2)7 at (245.1, 38.1)
- removed the D1(2)8 at (245.1, 129.5)
- removed the D1(2)9 at (245.1, 83.8)
- removed the J1 at (211.5, 163.2)
- removed the J10 at (211.5, 87.0)
- removed the J3 at (211.5, 71.8)
- removed the J4 at (211.5, 117.5)
- removed the J5 at (211.5, 56.5)
- removed the J6 at (211.5, 148.0)
- removed the J7 at (211.5, 102.2)
- removed the J8 at (211.5, 41.3)
- removed the J9 at (211.5, 132.7)
- removed the P1 at (173.4, 111.1)
- removed the P10 at (173.4, 106.0)
- removed the P11 at (173.4, 98.4)
- removed the P3 at (181.0, 163.2)
- removed the P4 at (173.4, 95.9)
- removed the P5 at (173.4, 103.5)
- removed the P6 at (173.4, 93.3)
- removed the P7 at (173.4, 108.6)
- removed the P8 at (173.4, 101.0)
- removed the P9 at (173.4, 90.8)
- removed the Q1 at (206.4, 160.7)
- removed the Q10 at (206.4, 145.4)
- removed the Q11 at (200.0, 99.7)
- removed the Q12 at (206.4, 99.7)
- removed the Q13 at (200.0, 38.7)
- removed the Q14 at (206.4, 38.7)
- removed the Q15 at (200.0, 130.2)
- removed the Q16 at (206.4, 130.2)
- removed the Q17 at (200.0, 84.5)
- removed the Q18 at (206.4, 84.5)
- removed the Q2 at (200.0, 160.7)
- removed the Q3 at (200.0, 69.2)
- removed the Q4 at (206.4, 69.2)
- removed the Q5 at (200.0, 114.9)
- removed the Q6 at (206.4, 114.9)
- removed the Q7 at (200.0, 54.0)
- removed the Q8 at (206.4, 54.0)
- removed the Q9 at (200.0, 145.4)
- removed the R10 at (239.4, 67.9)
- removed the R11 at (239.4, 113.7)
- removed the R12 at (195.2, 57.8)
- removed the R13 at (195.2, 149.2)
- removed the R14 at (195.2, 103.5)
- removed the R15 at (231.8, 58.4)
- removed the R16 at (231.8, 149.7)
- removed the R17 at (231.8, 104.1)
- removed the R18 at (239.4, 52.7)
- removed the R19 at (239.4, 144.1)
- removed the R2 at (231.8, 165.1)
- removed the R20 at (239.4, 98.4)
- removed the R21 at (195.2, 42.5)
- removed the R22 at (195.2, 134.0)
- removed the R23 at (195.2, 88.3)
- removed the R24 at (231.8, 43.2)
- removed the R25 at (231.8, 134.6)
- removed the R26 at (231.8, 88.9)
- removed the R27 at (239.4, 37.5)
- removed the R28 at (239.4, 128.9)
- removed the R29 at (239.4, 83.2)
- removed the R3 at (239.4, 159.4)
- removed the R4 at (195.2, 164.5)
- removed the R6 at (195.2, 73.0)
- removed the R7 at (195.2, 118.7)
- removed the R8 at (231.8, 73.7)
- removed the R9 at (231.8, 119.4)
- moved Q13 111.9 mm to (170.8, 74.9), turned to 180 degrees
- moved R21 110.2 mm to (167.0, 70.1), turned to 90 degrees
- moved Q14 108.5 mm to (170.8, 81.3), turned to 180 degrees
- moved D1(2)7 104.3 mm to (171.4, 120.0), turned to 0 degrees
- moved R27 104.1 mm to (172.1, 114.3), turned to 90 degrees
- moved P3 104.1 mm to (46.4, 55.9), turned to 180 degrees
- moved J8 102.8 mm to (168.3, 86.4), turned to 0 degrees
- moved R24 95.6 mm to (166.4, 106.7), turned to 270 degrees
- moved Q7 92.7 mm to (155.6, 74.9), turned to 180 degrees
- moved R4 92.6 mm to (45.1, 70.1), turned to 45 degrees
- moved R12 91.9 mm to (151.8, 70.1), turned to 90 degrees
- moved P9 88.6 mm to (118.7, 48.3), turned to 0 degrees
- moved Q8 88.6 mm to (155.6, 81.3), turned to 180 degrees
- moved P6 87.5 mm to (116.2, 48.3), turned to 0 degrees
- moved P4 86.6 mm to (113.7, 48.3), turned to 0 degrees
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Routing:
- net +5V: track 1444.8 -> 722.4 mm
- net -5V: track 1092.9 -> 546.5 mm
- net GNDREF: track 460.3 -> 230.1 mm
- net Net-(P9-Pad1): track 106.8 -> 53.4 mm
- net Net-(P1-Pad1): track 100.5 -> 50.3 mm
- net Net-(J3-Pad1): track 88.3 -> 44.1 mm
- net Net-(J4-Pad1): track 88.3 -> 44.1 mm
- net Net-(J5-Pad1): track 88.3 -> 44.1 mm
- net Net-(J7-Pad1): track 88.3 -> 44.1 mm
- net Net-(J9-Pad1): track 88.3 -> 44.1 mm
- net Net-(J1-Pad1): track 88.3 -> 44.1 mm
- net Net-(J6-Pad1): track 88.3 -> 44.1 mm
- net Net-(J8-Pad1): track 88.3 -> 44.1 mm
- net Net-(J10-Pad1): track 88.3 -> 44.1 mm
- net Net-(P6-Pad1): track 80.6 -> 40.3 mm
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