File: trimux/trimux.kicad_pcb (KiCad board)
At the start: 2 copper layers, 9 parts, among them IC1 DG403, IC2 DG403

Commit message: trimux
Parts:
- added ?: , trimux:SolderWirePad_single_0-8mmDrill, F.Cu at (52.1, 52.1)
- added ?: , trimux:SolderWirePad_single_0-8mmDrill, F.Cu at (40.6, 40.6)
- added ?: , trimux:SolderWirePad_single_0-8mmDrill, F.Cu at (39.4, 39.4)
- added ?: , trimux:SolderWirePad_single_0-8mmDrill, F.Cu at (38.1, 38.1)
- added ?: , trimux:SolderWirePad_single_0-8mmDrill, F.Cu at (36.8, 36.8)
- added ?: , trimux:SolderWirePad_single_0-8mmDrill, F.Cu at (35.6, 35.6)
- added ?: , trimux:SolderWirePad_single_0-8mmDrill, F.Cu at (34.3, 34.3)
- added ?: , trimux:SolderWirePad_single_0-8mmDrill, F.Cu at (33.0, 33.0)
- added ?: , trimux:SolderWirePad_single_0-8mmDrill, F.Cu at (31.8, 31.8)
- added ?: , trimux:SolderWirePad_single_0-8mmDrill, F.Cu at (30.5, 30.5)
- added ?: , trimux:SolderWirePad_single_0-8mmDrill, F.Cu at (29.2, 29.2)
- added ?: , trimux:SolderWirePad_single_0-8mmDrill, F.Cu at (50.8, 50.8)
- added ?: , trimux:SolderWirePad_single_0-8mmDrill, F.Cu at (27.9, 27.9)
- added ?: , trimux:SolderWirePad_single_0-8mmDrill, F.Cu at (26.7, 26.7)
- added ?: , trimux:SolderWirePad_single_0-8mmDrill, F.Cu at (25.4, 25.4)
- added ?: , trimux:SolderWirePad_single_0-8mmDrill, F.Cu at (24.1, 24.1)
- added ?: , trimux:SolderWirePad_single_0-8mmDrill, F.Cu at (49.5, 49.5)
- added ?: , trimux:SolderWirePad_single_0-8mmDrill, F.Cu at (48.3, 48.3)
- added ?: , trimux:SolderWirePad_single_0-8mmDrill, F.Cu at (47.0, 47.0)
- added ?: , trimux:SolderWirePad_single_0-8mmDrill, F.Cu at (45.7, 45.7)
- added ?: , trimux:SolderWirePad_single_0-8mmDrill, F.Cu at (44.5, 44.5)
- added ?: , trimux:SolderWirePad_single_0-8mmDrill, F.Cu at (43.2, 43.2)
- added ?: , trimux:SolderWirePad_single_0-8mmDrill, F.Cu at (41.9, 41.9)
- added C1: CP1, SMD_Packages:SMD-1206_Pol, F.Cu at (47.6, 38.4)
- added C2: CP1, SMD_Packages:SMD-1206_Pol, F.Cu at (48.3, 42.8)
- added C3: CP1, SMD_Packages:SMD-1206_Pol, F.Cu at (41.9, 33.9)
- added C4: CP1, SMD_Packages:SMD-1206_Pol, F.Cu at (46.4, 33.9)
- added IC1: DG403, SMD_Packages:SO-16-N, F.Cu at (55.9, 41.5)
- added IC2: DG403, SMD_Packages:SO-16-N, F.Cu at (43.2, 26.3)
- added JP1: CONN_01X05, Pin_Headers:Pin_Header_Straight_1x05, F.Cu at (61.0, 14.9)
- added JP2: CONN_01X05, Pin_Headers:Pin_Header_Straight_1x05, F.Cu at (45.7, 14.9)
- added JP3: CONN_01X03, Pin_Headers:Pin_Header_Straight_1x03, F.Cu at (30.5, 14.9)
- moved C4 10.6 mm to (29.8, 41.9)
- moved C3 10.5 mm to (34.3, 41.9)
- moved C2 10.2 mm to (27.9, 33.0), turned to 180 degrees
- moved C1 7.67 mm to (28.6, 37.5), turned to 0 degrees
- moved IC2 6.48 mm to (33.0, 49.5), turned to 0 degrees
- moved IC1 1.80 mm to (20.3, 34.3)
Routing:
- net (no net): track 727.3 -> 0.00 mm, vias 13 -> 0
- net /V-NEG: track 0.00 -> 150.4 mm, vias 0 -> 6
- net /S1: track 0.00 -> 147.5 mm, vias 0 -> 6
- net /V-POS: track 0.00 -> 129.7 mm, vias 0 -> 8
- net /S2: track 0.00 -> 125.1 mm, vias 0 -> 4
- net /GND: track 0.00 -> 111.8 mm, vias 0 -> 2
- net /C2: track 0.00 -> 110.8 mm, vias 0 -> 4
- net /O1: track 0.00 -> 101.7 mm, vias 0 -> 4
- net /N2: track 0.00 -> 88.4 mm, vias 0 -> 4
- net /C1: track 0.00 -> 84.3 mm, vias 0 -> 2
- net /P1: track 0.00 -> 76.6 mm, vias 0 -> 4
- net Net-(IC1-Pad16): track 0.00 -> 70.9 mm
- net /N1: track 0.00 -> 70.5 mm, vias 0 -> 2
- net Net-(IC1-Pad9): track 0.00 -> 60.4 mm
- net /P2: track 0.00 -> 48.7 mm, vias 0 -> 2
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Other:
- board outline added: 50 x 50.3 mm
- net class Default: via_drill 0.4 -> 0.5
- net class Power lines: via_drill 0.4 -> 0.8
- board text added: "-5 0 5"
- board text added: "S N O P C"

Commit message: trimux
Parts:
- removed the C1 at (47.6, 38.4)
- removed the C2 at (48.3, 42.8)
- removed the C3 at (41.9, 33.9)
- removed the C4 at (46.4, 33.9)
- removed the IC1 at (55.9, 41.5)
- removed the IC2 at (43.2, 26.3)
- removed the JP1 at (61.0, 14.9)
- removed the JP2 at (45.7, 14.9)
- removed the JP3 at (30.5, 14.9)
- added ?: , trimux:SolderWirePad_single_0-8mmDrill, F.Cu at (184.2, 27.3)
- added ?: , trimux:SolderWirePad_single_0-8mmDrill, F.Cu at (195.6, 38.7)
- added ?: , trimux:SolderWirePad_single_0-8mmDrill, F.Cu at (195.6, 152.4)
- added ?: , trimux:SolderWirePad_single_0-8mmDrill, F.Cu at (196.8, 153.7)
- added ?: , trimux:SolderWirePad_single_0-8mmDrill, F.Cu at (198.1, 154.9)
- added ?: , trimux:SolderWirePad_single_0-8mmDrill, F.Cu at (199.4, 156.2)
- added ?: , trimux:SolderWirePad_single_0-8mmDrill, F.Cu at (200.7, 157.5)
- added ?: , trimux:SolderWirePad_single_0-8mmDrill, F.Cu at (201.9, 158.8)
- added ?: , trimux:SolderWirePad_single_0-8mmDrill, F.Cu at (203.2, 160.0)
- added ?: , trimux:SolderWirePad_single_0-8mmDrill, F.Cu at (204.5, 161.3)
- added ?: , trimux:SolderWirePad_single_0-8mmDrill, F.Cu at (205.7, 162.6)
- added ?: , trimux:SolderWirePad_single_0-8mmDrill, F.Cu at (207.0, 163.8)
- added ?: , trimux:SolderWirePad_single_0-8mmDrill, F.Cu at (196.8, 40.0)
- added ?: , trimux:SolderWirePad_single_0-8mmDrill, F.Cu at (208.3, 165.1)
- added ?: , trimux:SolderWirePad_single_0-8mmDrill, F.Cu at (209.6, 166.4)
- added ?: , trimux:SolderWirePad_single_0-8mmDrill, F.Cu at (210.8, 167.6)
- added ?: , trimux:SolderWirePad_single_0-8mmDrill, F.Cu at (212.1, 168.9)
- added ?: , trimux:SolderWirePad_single_0-8mmDrill, F.Cu at (213.4, 170.2)
- added ?: , trimux:SolderWirePad_single_0-8mmDrill, F.Cu at (214.6, 171.4)
- added ?: , trimux:SolderWirePad_single_0-8mmDrill, F.Cu at (208.3, 153.7)
- added ?: , trimux:SolderWirePad_single_0-8mmDrill, F.Cu at (209.6, 154.9)
- added ?: , trimux:SolderWirePad_single_0-8mmDrill, F.Cu at (210.8, 156.2)
- added ?: , trimux:SolderWirePad_single_0-8mmDrill, F.Cu at (212.1, 157.5)
- added ?: , trimux:SolderWirePad_single_0-8mmDrill, F.Cu at (198.1, 41.3)
- added ?: , trimux:SolderWirePad_single_0-8mmDrill, F.Cu at (213.4, 158.8)
- added ?: , trimux:SolderWirePad_single_0-8mmDrill, F.Cu at (214.6, 160.0)
- added ?: , trimux:SolderWirePad_single_0-8mmDrill, F.Cu at (215.9, 161.3)
- added ?: , trimux:SolderWirePad_single_0-8mmDrill, F.Cu at (217.2, 162.6)
- added ?: , trimux:SolderWirePad_single_0-8mmDrill, F.Cu at (218.4, 163.8)
- added ?: , trimux:SolderWirePad_single_0-8mmDrill, F.Cu at (219.7, 165.1)
- added ?: , trimux:SolderWirePad_single_0-8mmDrill, F.Cu at (221.0, 166.4)
- added ?: , trimux:SolderWirePad_single_0-8mmDrill, F.Cu at (222.2, 167.6)
- added ?: , trimux:SolderWirePad_single_0-8mmDrill, F.Cu at (223.5, 168.9)
- added ?: , trimux:SolderWirePad_single_0-8mmDrill, F.Cu at (224.8, 170.2)
- added ?: , trimux:SolderWirePad_single_0-8mmDrill, F.Cu at (199.4, 42.5)
- added ?: , trimux:SolderWirePad_single_0-8mmDrill, F.Cu at (226.1, 171.4)
- added ?: , trimux:SolderWirePad_single_0-8mmDrill, F.Cu at (227.3, 172.7)
- added ?: , trimux:SolderWirePad_single_0-8mmDrill, F.Cu at (228.6, 174.0)
- added ?: , trimux:SolderWirePad_single_0-8mmDrill, F.Cu at (229.9, 175.3)
- added ?: , trimux:SolderWirePad_single_0-8mmDrill, F.Cu at (231.1, 176.5)
- added ?: , trimux:SolderWirePad_single_0-8mmDrill, F.Cu at (232.4, 177.8)
- added ?: , trimux:SolderWirePad_single_0-8mmDrill, F.Cu at (233.7, 179.1)
- added ?: , trimux:SolderWirePad_single_0-8mmDrill, F.Cu at (234.9, 180.3)
- added ?: , trimux:SolderWirePad_single_0-8mmDrill, F.Cu at (236.2, 181.6)
- added ?: , trimux:SolderWirePad_single_0-8mmDrill, F.Cu at (118.1, 181.0)
- added ?: , trimux:SolderWirePad_single_0-8mmDrill, F.Cu at (200.7, 43.8)
- added ?: , trimux:SolderWirePad_single_0-8mmDrill, F.Cu at (116.8, 179.7)
- added ?: , trimux:SolderWirePad_single_0-8mmDrill, F.Cu at (115.6, 178.4)
- added ?: , trimux:SolderWirePad_single_0-8mmDrill, F.Cu at (114.3, 177.2)
- added ?: , trimux:SolderWirePad_single_0-8mmDrill, F.Cu at (113.0, 175.9)
- added ?: , trimux:SolderWirePad_single_0-8mmDrill, F.Cu at (111.8, 174.6)
- added ?: , trimux:SolderWirePad_single_0-8mmDrill, F.Cu at (110.5, 173.4)
- added ?: , trimux:SolderWirePad_single_0-8mmDrill, F.Cu at (109.2, 172.1)
- added ?: , trimux:SolderWirePad_single_0-8mmDrill, F.Cu at (108.0, 170.8)
- added ?: , trimux:SolderWirePad_single_0-8mmDrill, F.Cu at (106.7, 169.5)
- added ?: , trimux:SolderWirePad_single_0-8mmDrill, F.Cu at (105.4, 168.3)
- added ?: , trimux:SolderWirePad_single_0-8mmDrill, F.Cu at (201.9, 45.1)
- added ?: , trimux:SolderWirePad_single_0-8mmDrill, F.Cu at (104.1, 167.0)
- added ?: , trimux:SolderWirePad_single_0-8mmDrill, F.Cu at (102.9, 165.7)
- added ?: , trimux:SolderWirePad_single_0-8mmDrill, F.Cu at (101.6, 164.5)
- added ?: , trimux:SolderWirePad_single_0-8mmDrill, F.Cu at (100.3, 163.2)
- added ?: , trimux:SolderWirePad_single_0-8mmDrill, F.Cu at (99.1, 161.9)
- added ?: , trimux:SolderWirePad_single_0-8mmDrill, F.Cu at (97.8, 160.7)
- added ?: , trimux:SolderWirePad_single_0-8mmDrill, F.Cu at (96.5, 159.4)
- added ?: , trimux:SolderWirePad_single_0-8mmDrill, F.Cu at (95.2, 158.1)
- added ?: , trimux:SolderWirePad_single_0-8mmDrill, F.Cu at (94.0, 156.8)
- added ?: , trimux:SolderWirePad_single_0-8mmDrill, F.Cu at (92.7, 155.6)
- added ?: , trimux:SolderWirePad_single_0-8mmDrill, F.Cu at (203.2, 46.4)
- added ?: , trimux:SolderWirePad_single_0-8mmDrill, F.Cu at (91.4, 154.3)
- added ?: , trimux:SolderWirePad_single_0-8mmDrill, F.Cu at (90.2, 153.0)
- added ?: , trimux:SolderWirePad_single_0-8mmDrill, F.Cu at (96.5, 170.8)
- added ?: , trimux:SolderWirePad_single_0-8mmDrill, F.Cu at (95.2, 169.5)
- added ?: , trimux:SolderWirePad_single_0-8mmDrill, F.Cu at (94.0, 168.3)
- added ?: , trimux:SolderWirePad_single_0-8mmDrill, F.Cu at (92.7, 167.0)
- added ?: , trimux:SolderWirePad_single_0-8mmDrill, F.Cu at (91.4, 165.7)
- added ?: , trimux:SolderWirePad_single_0-8mmDrill, F.Cu at (90.2, 164.5)
- added ?: , trimux:SolderWirePad_single_0-8mmDrill, F.Cu at (88.9, 163.2)
- added ?: , trimux:SolderWirePad_single_0-8mmDrill, F.Cu at (87.6, 161.9)
- added ?: , trimux:SolderWirePad_single_0-8mmDrill, F.Cu at (204.5, 47.6)
- added ?: , trimux:SolderWirePad_single_0-8mmDrill, F.Cu at (86.4, 160.7)
- added ?: , trimux:SolderWirePad_single_0-8mmDrill, F.Cu at (85.1, 159.4)
- added ?: , trimux:SolderWirePad_single_0-8mmDrill, F.Cu at (83.8, 158.1)
- added ?: , trimux:SolderWirePad_single_0-8mmDrill, F.Cu at (82.5, 156.8)
- added ?: , trimux:SolderWirePad_single_0-8mmDrill, F.Cu at (81.3, 155.6)
- added ?: , trimux:SolderWirePad_single_0-8mmDrill, F.Cu at (80.0, 154.3)
- added ?: , trimux:SolderWirePad_single_0-8mmDrill, F.Cu at (78.7, 153.0)
- added ?: , trimux:SolderWirePad_single_0-8mmDrill, F.Cu at (77.5, 151.8)
- added ?: , trimux:SolderWirePad_single_0-8mmDrill, F.Cu at (76.2, 150.5)
- added ?: , trimux:SolderWirePad_single_0-8mmDrill, F.Cu at (74.9, 149.2)
- added ?: , trimux:SolderWirePad_single_0-8mmDrill, F.Cu at (205.7, 48.9)
- added ?: , trimux:SolderWirePad_single_0-8mmDrill, F.Cu at (73.7, 148.0)
- added ?: , trimux:SolderWirePad_single_0-8mmDrill, F.Cu at (72.4, 146.7)
- added ?: , trimux:SolderWirePad_single_0-8mmDrill, F.Cu at (71.1, 145.4)
- added ?: , trimux:SolderWirePad_single_0-8mmDrill, F.Cu at (69.8, 144.1)
- added ?: , trimux:SolderWirePad_single_0-8mmDrill, F.Cu at (68.6, 142.9)
- added ?: , trimux:SolderWirePad_single_0-8mmDrill, F.Cu at (67.3, 85.7)
- added ?: , trimux:SolderWirePad_single_0-8mmDrill, F.Cu at (68.6, 87.0)
- added ?: , trimux:SolderWirePad_single_0-8mmDrill, F.Cu at (69.8, 88.3)
- added ?: , trimux:SolderWirePad_single_0-8mmDrill, F.Cu at (71.1, 89.5)
- added ?: , trimux:SolderWirePad_single_0-8mmDrill, F.Cu at (72.4, 90.8)
- added ?: , trimux:SolderWirePad_single_0-8mmDrill, F.Cu at (207.0, 50.2)
- added ?: , trimux:SolderWirePad_single_0-8mmDrill, F.Cu at (73.7, 92.1)
- added ?: , trimux:SolderWirePad_single_0-8mmDrill, F.Cu at (74.9, 93.3)
- added ?: , trimux:SolderWirePad_single_0-8mmDrill, F.Cu at (76.2, 94.6)
- added ?: , trimux:SolderWirePad_single_0-8mmDrill, F.Cu at (77.5, 95.9)
- added ?: , trimux:SolderWirePad_single_0-8mmDrill, F.Cu at (78.7, 97.2)
- added ?: , trimux:SolderWirePad_single_0-8mmDrill, F.Cu at (80.0, 98.4)
- added ?: , trimux:SolderWirePad_single_0-8mmDrill, F.Cu at (81.3, 99.7)
- added ?: , trimux:SolderWirePad_single_0-8mmDrill, F.Cu at (82.5, 101.0)
- added ?: , trimux:SolderWirePad_single_0-8mmDrill, F.Cu at (83.8, 102.2)
- added ?: , trimux:SolderWirePad_single_0-8mmDrill, F.Cu at (85.1, 103.5)
- added ?: , trimux:SolderWirePad_single_0-8mmDrill, F.Cu at (185.4, 28.6)
- added ?: , trimux:SolderWirePad_single_0-8mmDrill, F.Cu at (208.3, 51.4)
- added ?: , trimux:SolderWirePad_single_0-8mmDrill, F.Cu at (86.4, 104.8)
- added ?: , trimux:SolderWirePad_single_0-8mmDrill, F.Cu at (87.6, 106.0)
- added ?: , trimux:SolderWirePad_single_0-8mmDrill, F.Cu at (88.9, 107.3)
- added ?: , trimux:SolderWirePad_single_0-8mmDrill, F.Cu at (90.2, 108.6)
- added ?: , trimux:SolderWirePad_single_0-8mmDrill, F.Cu at (91.4, 109.9)
- added ?: , trimux:SolderWirePad_single_0-8mmDrill, F.Cu at (92.7, 111.1)
- added ?: , trimux:SolderWirePad_single_0-8mmDrill, F.Cu at (94.0, 112.4)
- added ?: , trimux:SolderWirePad_single_0-8mmDrill, F.Cu at (95.2, 113.7)
- added ?: , trimux:SolderWirePad_single_0-8mmDrill, F.Cu at (88.9, 95.9)
- added ?: , trimux:SolderWirePad_single_0-8mmDrill, F.Cu at (90.2, 97.2)
- added ?: , trimux:SolderWirePad_single_0-8mmDrill, F.Cu at (209.6, 52.7)
- added ?: , trimux:SolderWirePad_single_0-8mmDrill, F.Cu at (91.4, 98.4)
- added ?: , trimux:SolderWirePad_single_0-8mmDrill, F.Cu at (92.7, 99.7)
- added ?: , trimux:SolderWirePad_single_0-8mmDrill, F.Cu at (94.0, 101.0)
- added ?: , trimux:SolderWirePad_single_0-8mmDrill, F.Cu at (95.2, 102.2)
- added ?: , trimux:SolderWirePad_single_0-8mmDrill, F.Cu at (96.5, 103.5)
- added ?: , trimux:SolderWirePad_single_0-8mmDrill, F.Cu at (97.8, 104.8)
- added ?: , trimux:SolderWirePad_single_0-8mmDrill, F.Cu at (99.1, 106.0)
- added ?: , trimux:SolderWirePad_single_0-8mmDrill, F.Cu at (100.3, 107.3)
- added ?: , trimux:SolderWirePad_single_0-8mmDrill, F.Cu at (101.6, 108.6)
- added ?: , trimux:SolderWirePad_single_0-8mmDrill, F.Cu at (102.9, 109.9)
- added ?: , trimux:SolderWirePad_single_0-8mmDrill, F.Cu at (210.8, 54.0)
- added ?: , trimux:SolderWirePad_single_0-8mmDrill, F.Cu at (104.1, 111.1)
- added ?: , trimux:SolderWirePad_single_0-8mmDrill, F.Cu at (105.4, 112.4)
- added ?: , trimux:SolderWirePad_single_0-8mmDrill, F.Cu at (106.7, 113.7)
- added ?: , trimux:SolderWirePad_single_0-8mmDrill, F.Cu at (108.0, 114.9)
- added ?: , trimux:SolderWirePad_single_0-8mmDrill, F.Cu at (109.2, 116.2)
- added ?: , trimux:SolderWirePad_single_0-8mmDrill, F.Cu at (110.5, 117.5)
- added ?: , trimux:SolderWirePad_single_0-8mmDrill, F.Cu at (111.8, 118.7)
- added ?: , trimux:SolderWirePad_single_0-8mmDrill, F.Cu at (113.0, 120.0)
- added ?: , trimux:SolderWirePad_single_0-8mmDrill, F.Cu at (114.3, 121.3)
- added ?: , trimux:SolderWirePad_single_0-8mmDrill, F.Cu at (115.6, 122.6)
- added ?: , trimux:SolderWirePad_single_0-8mmDrill, F.Cu at (212.1, 55.2)
- added ?: , trimux:SolderWirePad_single_0-8mmDrill, F.Cu at (116.8, 123.8)
- added ?: , trimux:SolderWirePad_single_0-8mmDrill, F.Cu at (115.6, 64.8)
- added ?: , trimux:SolderWirePad_single_0-8mmDrill, F.Cu at (114.3, 63.5)
- added ?: , trimux:SolderWirePad_single_0-8mmDrill, F.Cu at (113.0, 62.2)
- added ?: , trimux:SolderWirePad_single_0-8mmDrill, F.Cu at (111.8, 61.0)
- added ?: , trimux:SolderWirePad_single_0-8mmDrill, F.Cu at (110.5, 59.7)
- added ?: , trimux:SolderWirePad_single_0-8mmDrill, F.Cu at (109.2, 58.4)
- added ?: , trimux:SolderWirePad_single_0-8mmDrill, F.Cu at (108.0, 57.1)
- added ?: , trimux:SolderWirePad_single_0-8mmDrill, F.Cu at (106.7, 55.9)
- added ?: , trimux:SolderWirePad_single_0-8mmDrill, F.Cu at (105.4, 54.6)
- added ?: , trimux:SolderWirePad_single_0-8mmDrill, F.Cu at (205.7, 37.5)
- added ?: , trimux:SolderWirePad_single_0-8mmDrill, F.Cu at (104.1, 53.3)
- added ?: , trimux:SolderWirePad_single_0-8mmDrill, F.Cu at (102.9, 52.1)
- added ?: , trimux:SolderWirePad_single_0-8mmDrill, F.Cu at (101.6, 50.8)
- added ?: , trimux:SolderWirePad_single_0-8mmDrill, F.Cu at (100.3, 49.5)
- added ?: , trimux:SolderWirePad_single_0-8mmDrill, F.Cu at (99.1, 48.3)
- added ?: , trimux:SolderWirePad_single_0-8mmDrill, F.Cu at (97.8, 47.0)
- added ?: , trimux:SolderWirePad_single_0-8mmDrill, F.Cu at (96.5, 45.7)
- added ?: , trimux:SolderWirePad_single_0-8mmDrill, F.Cu at (95.2, 44.5)
- added ?: , trimux:SolderWirePad_single_0-8mmDrill, F.Cu at (94.0, 43.2)
- added ?: , trimux:SolderWirePad_single_0-8mmDrill, F.Cu at (92.7, 41.9)
- added ?: , trimux:SolderWirePad_single_0-8mmDrill, F.Cu at (207.0, 38.7)
- added ?: , trimux:SolderWirePad_single_0-8mmDrill, F.Cu at (91.4, 40.6)
- added ?: , trimux:SolderWirePad_single_0-8mmDrill, F.Cu at (90.2, 39.4)
- added ?: , trimux:SolderWirePad_single_0-8mmDrill, F.Cu at (88.9, 38.1)
- added ?: , trimux:SolderWirePad_single_0-8mmDrill, F.Cu at (87.6, 36.8)
- added ?: , trimux:SolderWirePad_single_0-8mmDrill, F.Cu at (208.3, 40.0)
- added ?: , trimux:SolderWirePad_single_0-8mmDrill, F.Cu at (209.6, 41.3)
- added ?: , trimux:SolderWirePad_single_0-8mmDrill, F.Cu at (210.8, 42.5)
- added ?: , trimux:SolderWirePad_single_0-8mmDrill, F.Cu at (212.1, 43.8)
- added ?: , trimux:SolderWirePad_single_0-8mmDrill, F.Cu at (186.7, 29.8)
- added ?: , trimux:SolderWirePad_single_0-8mmDrill, F.Cu at (213.4, 45.1)
- added ?: , trimux:SolderWirePad_single_0-8mmDrill, F.Cu at (214.6, 46.4)
- added ?: , trimux:SolderWirePad_single_0-8mmDrill, F.Cu at (215.9, 47.6)
- added ?: , trimux:SolderWirePad_single_0-8mmDrill, F.Cu at (217.2, 48.9)
- added ?: , trimux:SolderWirePad_single_0-8mmDrill, F.Cu at (218.4, 50.2)
- added ?: , trimux:SolderWirePad_single_0-8mmDrill, F.Cu at (219.7, 51.4)
- added ?: , trimux:SolderWirePad_single_0-8mmDrill, F.Cu at (221.0, 52.7)
- added ?: , trimux:SolderWirePad_single_0-8mmDrill, F.Cu at (222.2, 54.0)
- added ?: , trimux:SolderWirePad_single_0-8mmDrill, F.Cu at (223.5, 55.2)
- added ?: , trimux:SolderWirePad_single_0-8mmDrill, F.Cu at (224.8, 56.5)
- added ?: , trimux:SolderWirePad_single_0-8mmDrill, F.Cu at (188.0, 31.1)
- added ?: , trimux:SolderWirePad_single_0-8mmDrill, F.Cu at (226.1, 57.8)
- added ?: , trimux:SolderWirePad_single_0-8mmDrill, F.Cu at (227.3, 59.1)
- added ?: , trimux:SolderWirePad_single_0-8mmDrill, F.Cu at (228.6, 60.3)
- added ?: , trimux:SolderWirePad_single_0-8mmDrill, F.Cu at (229.9, 61.6)
- added ?: , trimux:SolderWirePad_single_0-8mmDrill, F.Cu at (231.1, 62.9)
- added ?: , trimux:SolderWirePad_single_0-8mmDrill, F.Cu at (232.4, 64.1)
- added ?: , trimux:SolderWirePad_single_0-8mmDrill, F.Cu at (233.7, 65.4)
- added ?: , trimux:SolderWirePad_single_0-8mmDrill, F.Cu at (234.9, 124.5)
- added ?: , trimux:SolderWirePad_single_0-8mmDrill, F.Cu at (233.7, 123.2)
- added ?: , trimux:SolderWirePad_single_0-8mmDrill, F.Cu at (232.4, 121.9)
- added ?: , trimux:SolderWirePad_single_0-8mmDrill, F.Cu at (189.2, 32.4)
- added ?: , trimux:SolderWirePad_single_0-8mmDrill, F.Cu at (231.1, 120.7)
- added ?: , trimux:SolderWirePad_single_0-8mmDrill, F.Cu at (229.9, 119.4)
- added ?: , trimux:SolderWirePad_single_0-8mmDrill, F.Cu at (228.6, 118.1)
- added ?: , trimux:SolderWirePad_single_0-8mmDrill, F.Cu at (227.3, 116.8)
- added ?: , trimux:SolderWirePad_single_0-8mmDrill, F.Cu at (226.1, 115.6)
- added ?: , trimux:SolderWirePad_single_0-8mmDrill, F.Cu at (224.8, 114.3)
- added ?: , trimux:SolderWirePad_single_0-8mmDrill, F.Cu at (223.5, 113.0)
- added ?: , trimux:SolderWirePad_single_0-8mmDrill, F.Cu at (222.2, 111.8)
- added ?: , trimux:SolderWirePad_single_0-8mmDrill, F.Cu at (221.0, 110.5)
- added ?: , trimux:SolderWirePad_single_0-8mmDrill, F.Cu at (219.7, 109.2)
- added ?: , trimux:SolderWirePad_single_0-8mmDrill, F.Cu at (190.5, 33.7)
- added ?: , trimux:SolderWirePad_single_0-8mmDrill, F.Cu at (218.4, 108.0)
- added ?: , trimux:SolderWirePad_single_0-8mmDrill, F.Cu at (217.2, 106.7)
- added ?: , trimux:SolderWirePad_single_0-8mmDrill, F.Cu at (215.9, 105.4)
- added ?: , trimux:SolderWirePad_single_0-8mmDrill, F.Cu at (214.6, 104.1)
- added ?: , trimux:SolderWirePad_single_0-8mmDrill, F.Cu at (213.4, 102.9)
- added ?: , trimux:SolderWirePad_single_0-8mmDrill, F.Cu at (212.1, 101.6)
- added ?: , trimux:SolderWirePad_single_0-8mmDrill, F.Cu at (210.8, 100.3)
- added ?: , trimux:SolderWirePad_single_0-8mmDrill, F.Cu at (209.6, 99.1)
- added ?: , trimux:SolderWirePad_single_0-8mmDrill, F.Cu at (208.3, 97.8)
- added ?: , trimux:SolderWirePad_single_0-8mmDrill, F.Cu at (207.0, 96.5)
- added ?: , trimux:SolderWirePad_single_0-8mmDrill, F.Cu at (191.8, 34.9)
- added ?: , trimux:SolderWirePad_single_0-8mmDrill, F.Cu at (213.4, 114.3)
- added ?: , trimux:SolderWirePad_single_0-8mmDrill, F.Cu at (212.1, 113.0)
- added ?: , trimux:SolderWirePad_single_0-8mmDrill, F.Cu at (210.8, 111.8)
- added ?: , trimux:SolderWirePad_single_0-8mmDrill, F.Cu at (209.6, 110.5)
- added ?: , trimux:SolderWirePad_single_0-8mmDrill, F.Cu at (208.3, 109.2)
- added ?: , trimux:SolderWirePad_single_0-8mmDrill, F.Cu at (207.0, 108.0)
- added ?: , trimux:SolderWirePad_single_0-8mmDrill, F.Cu at (205.7, 106.7)
- added ?: , trimux:SolderWirePad_single_0-8mmDrill, F.Cu at (204.5, 105.4)
- added ?: , trimux:SolderWirePad_single_0-8mmDrill, F.Cu at (203.2, 104.1)
- added ?: , trimux:SolderWirePad_single_0-8mmDrill, F.Cu at (201.9, 102.9)
- added ?: , trimux:SolderWirePad_single_0-8mmDrill, F.Cu at (193.0, 36.2)
- added ?: , trimux:SolderWirePad_single_0-8mmDrill, F.Cu at (200.7, 101.6)
- added ?: , trimux:SolderWirePad_single_0-8mmDrill, F.Cu at (199.4, 100.3)
- added ?: , trimux:SolderWirePad_single_0-8mmDrill, F.Cu at (198.1, 99.1)
- added ?: , trimux:SolderWirePad_single_0-8mmDrill, F.Cu at (196.8, 97.8)
- added ?: , trimux:SolderWirePad_single_0-8mmDrill, F.Cu at (195.6, 96.5)
- added ?: , trimux:SolderWirePad_single_0-8mmDrill, F.Cu at (194.3, 95.2)
- added ?: , trimux:SolderWirePad_single_0-8mmDrill, F.Cu at (193.0, 94.0)
- added ?: , trimux:SolderWirePad_single_0-8mmDrill, F.Cu at (191.8, 92.7)
- added ?: , trimux:SolderWirePad_single_0-8mmDrill, F.Cu at (190.5, 91.4)
- added ?: , trimux:SolderWirePad_single_0-8mmDrill, F.Cu at (189.2, 90.2)
- added ?: , trimux:SolderWirePad_single_0-8mmDrill, F.Cu at (194.3, 37.5)
- added ?: , trimux:SolderWirePad_single_0-8mmDrill, F.Cu at (188.0, 88.9)
- added ?: , trimux:SolderWirePad_single_0-8mmDrill, F.Cu at (186.7, 87.6)
- added ?: , trimux:SolderWirePad_single_0-8mmDrill, F.Cu at (185.4, 86.4)
- added ?: , trimux:SolderWirePad_single_0-8mmDrill, F.Cu at (186.7, 143.5)
- added ?: , trimux:SolderWirePad_single_0-8mmDrill, F.Cu at (188.0, 144.8)
- added ?: , trimux:SolderWirePad_single_0-8mmDrill, F.Cu at (189.2, 146.1)
- added ?: , trimux:SolderWirePad_single_0-8mmDrill, F.Cu at (190.5, 147.3)
- added ?: , trimux:SolderWirePad_single_0-8mmDrill, F.Cu at (191.8, 148.6)
- added ?: , trimux:SolderWirePad_single_0-8mmDrill, F.Cu at (193.0, 149.9)
- added ?: , trimux:SolderWirePad_single_0-8mmDrill, F.Cu at (194.3, 151.1)
- added C1: CP1, SMD_Packages:SMD-1206_Pol, F.Cu at (188.6, 40.6)
- added C1: CP1, SMD_Packages:SMD-1206_Pol, F.Cu at (112.4, 110.5)
- added C1: CP1, SMD_Packages:SMD-1206_Pol, F.Cu at (111.1, 51.4)
- added C1: CP1, SMD_Packages:SMD-1206_Pol, F.Cu at (229.2, 52.1)
- added C1: CP1, SMD_Packages:SMD-1206_Pol, F.Cu at (230.5, 111.1)
- added C1: CP1, SMD_Packages:SMD-1206_Pol, F.Cu at (189.9, 99.7)
- added C1: CP1, SMD_Packages:SMD-1206_Pol, F.Cu at (191.1, 156.8)
- added C1: CP1, SMD_Packages:SMD-1206_Pol, F.Cu at (231.8, 168.3)
- added C1: CP1, SMD_Packages:SMD-1206_Pol, F.Cu at (113.7, 167.6)
- added C1: CP1, SMD_Packages:SMD-1206_Pol, F.Cu at (73.0, 156.2)
- added C1: CP1, SMD_Packages:SMD-1206_Pol, F.Cu at (71.8, 99.1)
- added C2: CP1, SMD_Packages:SMD-1206_Pol, F.Cu at (188.0, 36.2)
- added C2: CP1, SMD_Packages:SMD-1206_Pol, F.Cu at (113.0, 114.9)
- added C2: CP1, SMD_Packages:SMD-1206_Pol, F.Cu at (111.8, 55.9)
- added C2: CP1, SMD_Packages:SMD-1206_Pol, F.Cu at (229.9, 56.5)
- added C2: CP1, SMD_Packages:SMD-1206_Pol, F.Cu at (231.1, 115.6)
- added C2: CP1, SMD_Packages:SMD-1206_Pol, F.Cu at (189.2, 95.2)
- added C2: CP1, SMD_Packages:SMD-1206_Pol, F.Cu at (190.5, 152.4)
- added C2: CP1, SMD_Packages:SMD-1206_Pol, F.Cu at (232.4, 172.7)
- added C2: CP1, SMD_Packages:SMD-1206_Pol, F.Cu at (114.3, 172.1)
- added C2: CP1, SMD_Packages:SMD-1206_Pol, F.Cu at (72.4, 151.8)
- added C2: CP1, SMD_Packages:SMD-1206_Pol, F.Cu at (71.1, 94.6)
- added C3: CP1, SMD_Packages:SMD-1206_Pol, F.Cu at (194.3, 45.1)
- added C3: CP1, SMD_Packages:SMD-1206_Pol, F.Cu at (106.7, 106.0)
- added C3: CP1, SMD_Packages:SMD-1206_Pol, F.Cu at (105.4, 47.0)
- added C3: CP1, SMD_Packages:SMD-1206_Pol, F.Cu at (223.5, 47.6)
- added C3: CP1, SMD_Packages:SMD-1206_Pol, F.Cu at (224.8, 106.7)
- added C3: CP1, SMD_Packages:SMD-1206_Pol, F.Cu at (195.6, 104.1)
- added C3: CP1, SMD_Packages:SMD-1206_Pol, F.Cu at (196.8, 161.3)
- added C3: CP1, SMD_Packages:SMD-1206_Pol, F.Cu at (226.1, 163.8)
- added C3: CP1, SMD_Packages:SMD-1206_Pol, F.Cu at (108.0, 163.2)
- added C3: CP1, SMD_Packages:SMD-1206_Pol, F.Cu at (78.7, 160.7)
- added C3: CP1, SMD_Packages:SMD-1206_Pol, F.Cu at (77.5, 103.5)
- added C4: CP1, SMD_Packages:SMD-1206_Pol, F.Cu at (189.9, 45.1)
- added C4: CP1, SMD_Packages:SMD-1206_Pol, F.Cu at (111.1, 106.0)
- added C4: CP1, SMD_Packages:SMD-1206_Pol, F.Cu at (109.9, 47.0)
- added C4: CP1, SMD_Packages:SMD-1206_Pol, F.Cu at (228.0, 47.6)
- added C4: CP1, SMD_Packages:SMD-1206_Pol, F.Cu at (229.2, 106.7)
- added C4: CP1, SMD_Packages:SMD-1206_Pol, F.Cu at (191.1, 104.1)
- added C4: CP1, SMD_Packages:SMD-1206_Pol, F.Cu at (192.4, 161.3)
- added C4: CP1, SMD_Packages:SMD-1206_Pol, F.Cu at (230.5, 163.8)
- added C4: CP1, SMD_Packages:SMD-1206_Pol, F.Cu at (112.4, 163.2)
- added C4: CP1, SMD_Packages:SMD-1206_Pol, F.Cu at (74.3, 160.7)
- added C4: CP1, SMD_Packages:SMD-1206_Pol, F.Cu at (73.0, 103.5)
- added IC1: DG403, SMD_Packages:SO-16-N, F.Cu at (180.3, 37.5)
- added IC1: DG403, SMD_Packages:SO-16-N, F.Cu at (120.7, 113.7)
- added IC1: DG403, SMD_Packages:SO-16-N, F.Cu at (119.4, 54.6)
- added IC1: DG403, SMD_Packages:SO-16-N, F.Cu at (237.5, 55.2)
- added IC1: DG403, SMD_Packages:SO-16-N, F.Cu at (238.8, 114.3)
- added IC1: DG403, SMD_Packages:SO-16-N, F.Cu at (181.6, 96.5)
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Routing:
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Other:
- board size 50 x 50.3 mm -> 192.3 x 156.5 mm

Commit message: trimux
Parts:
- removed the ? at (184.2, 27.3)
- removed the ? at (195.6, 38.7)
- removed the ? at (195.6, 152.4)
- removed the ? at (196.8, 153.7)
- removed the ? at (198.1, 154.9)
- removed the ? at (199.4, 156.2)
- removed the ? at (200.7, 157.5)
- removed the ? at (201.9, 158.8)
- removed the ? at (203.2, 160.0)
- removed the ? at (204.5, 161.3)
- removed the ? at (205.7, 162.6)
- removed the ? at (207.0, 163.8)
- removed the ? at (196.8, 40.0)
- removed the ? at (208.3, 165.1)
- removed the ? at (209.6, 166.4)
- removed the ? at (210.8, 167.6)
- removed the ? at (212.1, 168.9)
- removed the ? at (213.4, 170.2)
- removed the ? at (214.6, 171.4)
- removed the ? at (208.3, 153.7)
- removed the ? at (209.6, 154.9)
- removed the ? at (210.8, 156.2)
- removed the ? at (212.1, 157.5)
- removed the ? at (198.1, 41.3)
- removed the ? at (213.4, 158.8)
- removed the ? at (214.6, 160.0)
- removed the ? at (215.9, 161.3)
- removed the ? at (217.2, 162.6)
- removed the ? at (218.4, 163.8)
- removed the ? at (219.7, 165.1)
- removed the ? at (221.0, 166.4)
- removed the ? at (222.2, 167.6)
- removed the ? at (223.5, 168.9)
- removed the ? at (224.8, 170.2)
- removed the ? at (199.4, 42.5)
- removed the ? at (226.1, 171.4)
- removed the ? at (227.3, 172.7)
- removed the ? at (228.6, 174.0)
- removed the ? at (229.9, 175.3)
- removed the ? at (231.1, 176.5)
- removed the ? at (232.4, 177.8)
- removed the ? at (233.7, 179.1)
- removed the ? at (234.9, 180.3)
- removed the ? at (236.2, 181.6)
- removed the ? at (118.1, 181.0)
- removed the ? at (200.7, 43.8)
- removed the ? at (116.8, 179.7)
- removed the ? at (115.6, 178.4)
- removed the ? at (114.3, 177.2)
- removed the ? at (113.0, 175.9)
- removed the ? at (111.8, 174.6)
- removed the ? at (110.5, 173.4)
- removed the ? at (109.2, 172.1)
- removed the ? at (108.0, 170.8)
- removed the ? at (106.7, 169.5)
- removed the ? at (105.4, 168.3)
- removed the ? at (201.9, 45.1)
- removed the ? at (104.1, 167.0)
- removed the ? at (102.9, 165.7)
- removed the ? at (101.6, 164.5)
- removed the ? at (100.3, 163.2)
- removed the ? at (99.1, 161.9)
- removed the ? at (97.8, 160.7)
- removed the ? at (96.5, 159.4)
- removed the ? at (95.2, 158.1)
- removed the ? at (94.0, 156.8)
- removed the ? at (92.7, 155.6)
- removed the ? at (203.2, 46.4)
- removed the ? at (91.4, 154.3)
- removed the ? at (90.2, 153.0)
- removed the ? at (96.5, 170.8)
- removed the ? at (95.2, 169.5)
- removed the ? at (94.0, 168.3)
- removed the ? at (92.7, 167.0)
- removed the ? at (91.4, 165.7)
- removed the ? at (90.2, 164.5)
- removed the ? at (88.9, 163.2)
- removed the ? at (87.6, 161.9)
- removed the ? at (204.5, 47.6)
- removed the ? at (86.4, 160.7)
- removed the ? at (85.1, 159.4)
- removed the ? at (83.8, 158.1)
- removed the ? at (82.5, 156.8)
- removed the ? at (81.3, 155.6)
- removed the ? at (80.0, 154.3)
- removed the ? at (78.7, 153.0)
- removed the ? at (77.5, 151.8)
- removed the ? at (76.2, 150.5)
- removed the ? at (74.9, 149.2)
- removed the ? at (205.7, 48.9)
- removed the ? at (73.7, 148.0)
- removed the ? at (72.4, 146.7)
- removed the ? at (71.1, 145.4)
- removed the ? at (69.8, 144.1)
- removed the ? at (68.6, 142.9)
- removed the ? at (67.3, 85.7)
- removed the ? at (68.6, 87.0)
- removed the ? at (69.8, 88.3)
- removed the ? at (71.1, 89.5)
- removed the ? at (72.4, 90.8)
- removed the ? at (207.0, 50.2)
- removed the ? at (73.7, 92.1)
- removed the ? at (74.9, 93.3)
- removed the ? at (76.2, 94.6)
- removed the ? at (77.5, 95.9)
- removed the ? at (78.7, 97.2)
- removed the ? at (80.0, 98.4)
- removed the ? at (81.3, 99.7)
- removed the ? at (82.5, 101.0)
- removed the ? at (83.8, 102.2)
- removed the ? at (85.1, 103.5)
- removed the ? at (185.4, 28.6)
- removed the ? at (208.3, 51.4)
- removed the ? at (86.4, 104.8)
- removed the ? at (87.6, 106.0)
- removed the ? at (88.9, 107.3)
- removed the ? at (90.2, 108.6)
- removed the ? at (91.4, 109.9)
- removed the ? at (92.7, 111.1)
- removed the ? at (94.0, 112.4)
- removed the ? at (95.2, 113.7)
- removed the ? at (88.9, 95.9)
- removed the ? at (90.2, 97.2)
- removed the ? at (209.6, 52.7)
- removed the ? at (91.4, 98.4)
- removed the ? at (92.7, 99.7)
- removed the ? at (94.0, 101.0)
- removed the ? at (95.2, 102.2)
- removed the ? at (96.5, 103.5)
- removed the ? at (97.8, 104.8)
- removed the ? at (99.1, 106.0)
- removed the ? at (100.3, 107.3)
- removed the ? at (101.6, 108.6)
- removed the ? at (102.9, 109.9)
- removed the ? at (210.8, 54.0)
- removed the ? at (104.1, 111.1)
- removed the ? at (105.4, 112.4)
- removed the ? at (106.7, 113.7)
- removed the ? at (108.0, 114.9)
- removed the ? at (109.2, 116.2)
- removed the ? at (110.5, 117.5)
- removed the ? at (111.8, 118.7)
- removed the ? at (113.0, 120.0)
- removed the ? at (114.3, 121.3)
- removed the ? at (115.6, 122.6)
- removed the ? at (212.1, 55.2)
- removed the ? at (116.8, 123.8)
- removed the ? at (115.6, 64.8)
- removed the ? at (114.3, 63.5)
- removed the ? at (113.0, 62.2)
- removed the ? at (111.8, 61.0)
- removed the ? at (110.5, 59.7)
- removed the ? at (109.2, 58.4)
- removed the ? at (108.0, 57.1)
- removed the ? at (106.7, 55.9)
- removed the ? at (105.4, 54.6)
- removed the ? at (205.7, 37.5)
- removed the ? at (104.1, 53.3)
- removed the ? at (102.9, 52.1)
- removed the ? at (101.6, 50.8)
- removed the ? at (100.3, 49.5)
- removed the ? at (99.1, 48.3)
- removed the ? at (97.8, 47.0)
- removed the ? at (96.5, 45.7)
- removed the ? at (95.2, 44.5)
- removed the ? at (94.0, 43.2)
- removed the ? at (92.7, 41.9)
- removed the ? at (207.0, 38.7)
- removed the ? at (91.4, 40.6)
- removed the ? at (90.2, 39.4)
- removed the ? at (88.9, 38.1)
- removed the ? at (87.6, 36.8)
- removed the ? at (208.3, 40.0)
- removed the ? at (209.6, 41.3)
- removed the ? at (210.8, 42.5)
- removed the ? at (212.1, 43.8)
- removed the ? at (186.7, 29.8)
- removed the ? at (213.4, 45.1)
- removed the ? at (214.6, 46.4)
- removed the ? at (215.9, 47.6)
- removed the ? at (217.2, 48.9)
- removed the ? at (218.4, 50.2)
- removed the ? at (219.7, 51.4)
- removed the ? at (221.0, 52.7)
- removed the ? at (222.2, 54.0)
- removed the ? at (223.5, 55.2)
- removed the ? at (224.8, 56.5)
- removed the ? at (188.0, 31.1)
- removed the ? at (226.1, 57.8)
- removed the ? at (227.3, 59.1)
- removed the ? at (228.6, 60.3)
- removed the ? at (229.9, 61.6)
- removed the ? at (231.1, 62.9)
- removed the ? at (232.4, 64.1)
- removed the ? at (233.7, 65.4)
- removed the ? at (234.9, 124.5)
- removed the ? at (233.7, 123.2)
- removed the ? at (232.4, 121.9)
- removed the ? at (189.2, 32.4)
- removed the ? at (231.1, 120.7)
- removed the ? at (229.9, 119.4)
- removed the ? at (228.6, 118.1)
- removed the ? at (227.3, 116.8)
- removed the ? at (226.1, 115.6)
- removed the ? at (224.8, 114.3)
- removed the ? at (223.5, 113.0)
- removed the ? at (222.2, 111.8)
- removed the ? at (221.0, 110.5)
- removed the ? at (219.7, 109.2)
- removed the ? at (190.5, 33.7)
- removed the ? at (218.4, 108.0)
- removed the ? at (217.2, 106.7)
- removed the ? at (215.9, 105.4)
- removed the ? at (214.6, 104.1)
- removed the ? at (213.4, 102.9)
- removed the ? at (212.1, 101.6)
- removed the ? at (210.8, 100.3)
- removed the ? at (209.6, 99.1)
- removed the ? at (208.3, 97.8)
- removed the ? at (207.0, 96.5)
- removed the ? at (191.8, 34.9)
- removed the ? at (213.4, 114.3)
- removed the ? at (212.1, 113.0)
- removed the ? at (210.8, 111.8)
- removed the ? at (209.6, 110.5)
- removed the ? at (208.3, 109.2)
- removed the ? at (207.0, 108.0)
- removed the ? at (205.7, 106.7)
- removed the ? at (204.5, 105.4)
- removed the ? at (203.2, 104.1)
- removed the ? at (201.9, 102.9)
- removed the ? at (193.0, 36.2)
- removed the ? at (200.7, 101.6)
- removed the ? at (199.4, 100.3)
- removed the ? at (198.1, 99.1)
- removed the ? at (196.8, 97.8)
- removed the ? at (195.6, 96.5)
- removed the ? at (194.3, 95.2)
- removed the ? at (193.0, 94.0)
- removed the ? at (191.8, 92.7)
- removed the ? at (190.5, 91.4)
- removed the ? at (189.2, 90.2)
- removed the ? at (194.3, 37.5)
- removed the ? at (188.0, 88.9)
- removed the ? at (186.7, 87.6)
- removed the ? at (185.4, 86.4)
- removed the ? at (186.7, 143.5)
- removed the ? at (188.0, 144.8)
- removed the ? at (189.2, 146.1)
- removed the ? at (190.5, 147.3)
- removed the ? at (191.8, 148.6)
- removed the ? at (193.0, 149.9)
- removed the ? at (194.3, 151.1)
- removed the C1 at (188.6, 40.6)
- removed the C1 at (112.4, 110.5)
- removed the C1 at (111.1, 51.4)
- removed the C1 at (229.2, 52.1)
- removed the C1 at (230.5, 111.1)
- removed the C1 at (189.9, 99.7)
- removed the C1 at (191.1, 156.8)
- removed the C1 at (231.8, 168.3)
- removed the C1 at (113.7, 167.6)
- removed the C1 at (73.0, 156.2)
- removed the C1 at (71.8, 99.1)
- removed the C2 at (188.0, 36.2)
- removed the C2 at (113.0, 114.9)
- removed the C2 at (111.8, 55.9)
- removed the C2 at (229.9, 56.5)
- removed the C2 at (231.1, 115.6)
- removed the C2 at (189.2, 95.2)
- removed the C2 at (190.5, 152.4)
- removed the C2 at (232.4, 172.7)
- removed the C2 at (114.3, 172.1)
- removed the C2 at (72.4, 151.8)
- removed the C2 at (71.1, 94.6)
- removed the C3 at (194.3, 45.1)
- removed the C3 at (106.7, 106.0)
- removed the C3 at (105.4, 47.0)
- removed the C3 at (223.5, 47.6)
- removed the C3 at (224.8, 106.7)
- removed the C3 at (195.6, 104.1)
- removed the C3 at (196.8, 161.3)
- removed the C3 at (226.1, 163.8)
- removed the C3 at (108.0, 163.2)
- removed the C3 at (78.7, 160.7)
- removed the C3 at (77.5, 103.5)
- removed the C4 at (189.9, 45.1)
- removed the C4 at (111.1, 106.0)
- removed the C4 at (109.9, 47.0)
- removed the C4 at (228.0, 47.6)
- removed the C4 at (229.2, 106.7)
- removed the C4 at (191.1, 104.1)
- removed the C4 at (192.4, 161.3)
- removed the C4 at (230.5, 163.8)
- removed the C4 at (112.4, 163.2)
- removed the C4 at (74.3, 160.7)
- removed the C4 at (73.0, 103.5)
- removed the IC1 at (180.3, 37.5)
- removed the IC1 at (120.7, 113.7)
- removed the IC1 at (119.4, 54.6)
- removed the IC1 at (237.5, 55.2)
- removed the IC1 at (238.8, 114.3)
- removed the IC1 at (181.6, 96.5)
- removed the IC1 at (182.9, 153.7)
- removed the IC1 at (240.0, 171.4)
- removed the IC1 at (121.9, 170.8)
- removed the IC1 at (64.8, 153.0)
- removed the IC1 at (63.5, 95.9)
- removed the IC2 at (193.0, 52.7)
- removed the IC2 at (108.0, 98.4)
- removed the IC2 at (106.7, 39.4)
- removed the IC2 at (224.8, 40.0)
- removed the IC2 at (226.1, 99.1)
- removed the IC2 at (194.3, 111.8)
- removed the IC2 at (195.6, 168.9)
- removed the IC2 at (227.3, 156.2)
- removed the IC2 at (109.2, 155.6)
- removed the IC2 at (77.5, 168.3)
- removed the IC2 at (76.2, 111.1)
- removed the JP1 at (175.3, 64.1)
- removed the JP1 at (125.7, 87.0)
- removed the JP1 at (124.5, 27.9)
- removed the JP1 at (242.6, 28.6)
- removed the JP1 at (243.8, 87.6)
- removed the JP1 at (176.5, 123.2)
- removed the JP1 at (177.8, 180.3)
- removed the JP1 at (245.1, 144.8)
- removed the JP1 at (127.0, 144.1)
- removed the JP1 at (59.7, 179.7)
- removed the JP1 at (58.4, 122.6)
- removed the JP2 at (190.5, 64.1)
- removed the JP2 at (110.5, 87.0)
- removed the JP2 at (109.2, 27.9)
- removed the JP2 at (227.3, 28.6)
- removed the JP2 at (228.6, 87.6)
- removed the JP2 at (191.8, 123.2)
- removed the JP2 at (193.0, 180.3)
- removed the JP2 at (229.9, 144.8)
- removed the JP2 at (111.8, 144.1)
- removed the JP2 at (74.9, 179.7)
- removed the JP2 at (73.7, 122.6)
- removed the JP3 at (205.7, 64.1)
- removed the JP3 at (95.2, 87.0)
- removed the JP3 at (94.0, 27.9)
- removed the JP3 at (212.1, 28.6)
- removed the JP3 at (213.4, 87.6)
- removed the JP3 at (207.0, 123.2)
- removed the JP3 at (208.3, 180.3)
- removed the JP3 at (214.6, 144.8)
- removed the JP3 at (96.5, 144.1)
- removed the JP3 at (90.2, 179.7)
- removed the JP3 at (88.9, 122.6)
- added C1: CP1, SMD_Packages:SMD-1206_Pol, F.Cu at (88.4, 74.1)
- added C2: CP1, SMD_Packages:SMD-1206_Pol, F.Cu at (89.0, 78.5)
- added C3: CP1, SMD_Packages:SMD-1206_Pol, F.Cu at (82.7, 69.7)
- added C4: CP1, SMD_Packages:SMD-1206_Pol, F.Cu at (87.1, 69.7)
- added IC1: DG403, SMD_Packages:SO-16-N, F.Cu at (96.6, 77.3)
- added IC2: DG403, SMD_Packages:SO-16-N, F.Cu at (83.9, 62.0)
- added JP1: CONN_01X05, Pin_Headers:Pin_Header_Straight_1x05, F.Cu at (101.7, 50.6)
- added JP2: CONN_01X05, Pin_Headers:Pin_Header_Straight_1x05, F.Cu at (86.5, 50.6)
- added JP3: CONN_01X03, Pin_Headers:Pin_Header_Straight_1x03, F.Cu at (71.2, 50.6)
- moved ? 33.0 mm to (92.8, 87.6)
- moved ? 33.0 mm to (80.1, 74.9)
- moved ? 33.0 mm to (78.9, 73.6)
- moved ? 33.0 mm to (75.1, 69.8)
- moved ? 33.0 mm to (70.0, 64.7)
- moved ? 33.0 mm to (68.7, 63.4)
- moved ? 33.0 mm to (66.2, 60.9)
- moved ? 33.0 mm to (89.0, 83.8)
- moved ? 33.0 mm to (87.8, 82.5)
- moved ? 33.0 mm to (83.9, 78.7)
- moved IC1 33.0 mm to (61.1, 69.8)
- moved JP1 33.0 mm to (56.0, 96.5)
- moved JP2 33.0 mm to (71.2, 96.5)
- moved JP3 33.0 mm to (86.5, 96.5)
- moved ? 33.0 mm to (81.4, 76.1)
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Routing:
- net (no net): track 7555.5 -> 0.00 mm
- net /V-NEG: track 933.4 -> 155.6 mm, vias 36 -> 6
- net /S1: track 857.0 -> 142.8 mm, vias 36 -> 6
- net /V-POS: track 778.0 -> 129.7 mm, vias 48 -> 8
- net /C2: track 696.3 -> 116.1 mm, vias 24 -> 4
- net /GND: track 671.0 -> 111.8 mm, vias 12 -> 2
- net /S2: track 631.4 -> 105.2 mm, vias 12 -> 2
- net /O1: track 579.1 -> 96.5 mm, vias 24 -> 4
- net /N2: track 527.7 -> 87.9 mm, vias 24 -> 4
- net /C1: track 520.2 -> 86.7 mm, vias 12 -> 2
- net /N1: track 422.8 -> 70.5 mm, vias 12 -> 2
- net Net-(IC1-Pad16): track 419.8 -> 70.0 mm
- net /P1: track 404.1 -> 67.4 mm, vias 24 -> 4
- net Net-(IC1-Pad9): track 348.7 -> 58.1 mm
- net /P2: track 282.5 -> 47.1 mm, vias 12 -> 2
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Other:
- board size 192.3 x 156.5 mm -> 50 x 49.9 mm
- board text added: "TRIMUXsmd"
- board text added: "v12.03.2017"

Commit message: half-adder
Parts:
- removed JP1, JP2: CONN_01X05, Pin_Headers:Pin_Header_Straight_1x05
- removed JP3: CONN_01X03, Pin_Headers:Pin_Header_Straight_1x03
- added ?: , trimux:SolderWirePad_single_0-8mmDrill, F.Cu at (96.6, 85.2)
- added ?: , trimux:SolderWirePad_single_0-8mmDrill, F.Cu at (61.1, 61.8)
- added PWR: CONN_01X03, Pin_Headers:Pin_Header_Straight_1x03, F.Cu at (71.2, 50.6)
- added mux1: CONN_01X05, Pin_Headers:Pin_Header_Straight_1x05, F.Cu at (101.7, 50.6)
- added mux2: CONN_01X05, Pin_Headers:Pin_Header_Straight_1x05, F.Cu at (86.5, 50.6)
- renumbered JP3 to PWR, JP1 to mux1, JP2 to mux2
Routing:
- net /S1: track 142.8 -> 140.7 mm
