File: trimux/counter/counter.sch (KiCad schematic (older format))
At the start: 33 parts, among them P1 CONN_01X03, P2 CONN_01X03, P3 CONN_01X02, P4 CONN_01X03, P5 CONN_01X03, U1 trimux, U2 trimux, U3 trimux, U4 trimux, U5 trimux

Commit message: counter board
Parts:
- added D1: LED_Dual_2pin, LEDs:LED-5MM, symbol LED_Dual_2pin-RESCUE-counter
- added P6: CONN_01X02, Pin_Headers:Pin_Header_Straight_1x02, symbol CONN_01X02
- added P7, P8, P9: CONN_01X03, Pin_Headers:Pin_Header_Straight_1x03, symbol CONN_01X03
- added R22: 1k, Resistors_SMD:R_1206_HandSoldering, symbol R
- added R23, R24, R25, R26, R27, R28, R29, R30, R31, R32, R33: 150, Resistors_SMD:R_1206_HandSoldering, symbol R
- added U6, U7: trimux, trimux:trimux1x15_2.54, symbol trimux
Connections:
- net +5V: now also P8.1 (P1), P9.1 (P1), R25.2, R27.2, R31.2, R33.2, U6.15 (+5V), U7.15 (+5V)
- net -5V: now also P8.3 (P3), P9.3 (P3), R23.2, R30.2, R32.2, U6.13 (-5V), U7.13 (-5V)
- net A: now also D1.2 (AK)
- net B: now also P7.1 (P1), R33.1
- net Cm: now also P7.3 (P3), U7.5 (C1)
- net Cs: now also P7.2 (P2), U7.11 (C2)
- net GNDREF: now also P8.2 (P2), P9.2 (P2), R22.2, R24.2, R26.2, R28.2, R29.2, U6.14 (0V), U7.14 (0V)
- new net: D1.1 (KA), R22.1
- new net: R31.1, U6.10 (P2)
- new net: U6.11 (C2), U7.8 (N2)
- new net: R23.1, U6.2 (N1)
- new net: R24.1, U6.3 (O1)
- new net: R26.1, U6.4 (P1)
- new net: U6.5 (C1), U7.2 (N1)
- new net: R28.1, U6.8 (N2)
- new net: R29.1, U6.9 (O2)
- new net: R32.1, U7.10 (P2)
- new net: R25.1, U7.3 (O1)
- new net: R27.1, U7.4 (P1)
- new net: R30.1, U7.9 (O2)
- new net ASSIGN: P6.1 (P1), U7.1 (S1), U7.7 (S2)
- new net CLK: P6.2 (P2), U6.1 (S1), U6.7 (S2)
