File: trimux/alu-a/alu-a.sch (KiCad schematic (older format))
At the start: 32 parts, among them J1 Conn_01x05, J10 Conn_01x05, J11 Conn_01x05, J2 Conn_01x01, J3 Conn_01x03, J4 Conn_01x01, J5 Conn_01x01, J6 Conn_01x01, J7 Conn_01x03, J8 Conn_01x05, J9 Conn_01x03, P1 CONN_01X03, P2 CONN_01X03, P3 CONN_01X03, U1 trimux, U10 trimux, U11 trimux, U12 trimux, U13 trimux, U2 trimux, U3 trimux, U4 trimux, U5 trimux, U6 trimux, U7 trimux, U8 trimux, U9 trimux

Commit message: alu-a routed
Parts:
- J2, J4, J5, J6: footprint (none) -> Pin_Headers:Pin_Header_Straight_1x01_Pitch2.54mm
- J3, J7, J9: footprint (none) -> Pin_Headers:Pin_Header_Straight_1x03_Pitch2.54mm
- R1: footprint (none) -> Resistors_SMD:R_1206_HandSoldering
Changed lines of the file:
@@
 F 0 "J7" H 2975 -2700 50  0000 C CNN
 F 1 "Conn_01x03" H 2975 -3100 50  0000 C CNN
-F 2 "" H 2975 -2900 50  0001 C CNN
+F 2 "Pin_Headers:Pin_Header_Straight_1x03_Pitch2.54mm" H 2975 -2900 50  0001 C CNN
 F 3 "" H 2975 -2900 50  0001 C CNN
 	1    2975 -2900
@@
 F 0 "R1" H 7505 -2080 50  0000 L CNN
 F 1 "10k" H 7505 -2140 50  0000 L CNN
-F 2 "" H 7475 -2100 50  0001 C CNN
+F 2 "Resistors_SMD:R_1206_HandSoldering" H 7475 -2100 50  0001 C CNN
 F 3 "" H 7475 -2100 50  0001 C CNN
 	1    7475 -2100
@@
 F 0 "J9" H 2975 -2150 50  0000 C CNN
 F 1 "Conn_01x03" H 2975 -2550 50  0000 C CNN
-F 2 "" H 2975 -2350 50  0001 C CNN
+F 2 "Pin_Headers:Pin_Header_Straight_1x03_Pitch2.54mm" H 2975 -2350 50  0001 C CNN
 F 3 "" H 2975 -2350 50  0001 C CNN
 	1    2975 -2350
@@
 F 0 "J3" H 2750 -1550 50  0000 C CNN
 F 1 "Conn_01x03" H 2750 -1950 50  0000 C CNN
-F 2 "" H 2750 -1750 50  0001 C CNN
+F 2 "Pin_Headers:Pin_Header_Straight_1x03_Pitch2.54mm" H 2750 -1750 50  0001 C CNN
 F 3 "" H 2750 -1750 50  0001 C CNN
 	1    2750 -1750
@@
 F 0 "J4" H 2750 -1200 50  0000 C CNN
 F 1 "Conn_01x01" H 2750 -1400 50  0000 C CNN
-F 2 "" H 2750 -1300 50  0001 C CNN
+F 2 "Pin_Headers:Pin_Header_Straight_1x01_Pitch2.54mm" H 2750 -1300 50  0001 C CNN
 F 3 "" H 2750 -1300 50  0001 C CNN
 	1    2750 -1300
@@
 F 0 "J2" H 2725 -875 50  0000 C CNN
 F 1 "Conn_01x01" H 2725 -1075 50  0000 C CNN
-F 2 "" H 2725 -975 50  0001 C CNN
+F 2 "Pin_Headers:Pin_Header_Straight_1x01_Pitch2.54mm" H 2725 -975 50  0001 C CNN
 F 3 "" H 2725 -975 50  0001 C CNN
 	1    2725 -975
@@
 F 0 "J5" H 2750 -550 50  0000 C CNN
 F 1 "Conn_01x01" H 2750 -750 50  0000 C CNN
-F 2 "" H 2750 -650 50  0001 C CNN
+F 2 "Pin_Headers:Pin_Header_Straight_1x01_Pitch2.54mm" H 2750 -650 50  0001 C CNN
 F 3 "" H 2750 -650 50  0001 C CNN
 	1    2750 -650
@@
 F 0 "J6" H 2750 -175 50  0000 C CNN
 F 1 "Conn_01x01" H 2750 -375 50  0000 C CNN
-F 2 "" H 2750 -275 50  0001 C CNN
+F 2 "Pin_Headers:Pin_Header_Straight_1x01_Pitch2.54mm" H 2750 -275 50  0001 C CNN
 F 3 "" H 2750 -275 50  0001 C CNN
 	1    2750 -275
